Commit message: pre project demo

File: multi_robot_follow/urdf/red_turtlebot.urdf (robot description, URDF)
Before this commit: robot red_turtlebot, 3 links, 2 joints
Links:
- removed link base_link
- removed link left_wheel
- removed link right_wheel
Joints:
- removed joint left_wheel_joint
- removed joint right_wheel_joint
